File: Projet_KICAD/Projet_PCBPolytech_git.kicad_sch (KiCad schematic)
At the start: 63 parts, among them J1 B2B-PH-K-S(LF)(SN), J12 USB_C_Receptacle_USB2.0_14P, J2 MOTOR_VIB, J3 Conn_01x14, J4 Conn_01x04, M1 LCM1027A2445F, Q1 AO3400A, U1 STM32F405RGTx, U2 CRYSTAL-SMD_2P-L5_0-W3_2, U3 SOP-8_L4_9-W3_9-P1_27-LS6_0-BL, U4 TLV62569DBV, U5 TPD2E2U06DCK, U6 SW-SMD_4P-L5_1-W5_1-P3_70-LS6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, U7 SW-SMD_4P-L5_1-W5_1-P3_70-LS6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

Commit message: ajout des broches USB
Connections:
- net TFT_MISO is gone; now on net TP_OUT: J3.9 (Pin_9)
- net TFT_MOSI is gone; now on net TP_DIN: J3.6 (Pin_6)
- net TFT_SCK is gone; now on net TP_CLK: J3.7 (Pin_7)
- net AUDIO_EN: now also U1.40 (PC9)
- net AUDIO_IN: now also U1.20 (PA4)
- net Detection_USB: now also U1.11 (PC3)
- net USB_D+: now also U1.45 (PA12)
- net USB_D-: now also U1.44 (PA11)
- no-connect marks 30 -> 25
Changed lines of the file:
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@@
-	)
-	(no_connect
-		(at 320.04 116.84)
 	)
 	(no_connect
@@
 	)
 	(no_connect
-		(at 360.68 99.06)
-	)
-	(no_connect
 		(at 320.04 121.92)
 	)
@@
 		(at 360.68 71.12)
 	)
-	(no_connect
-		(at 360.68 101.6)
-	)
-	(no_connect
-		(at 320.04 101.6)
-	)
-	(no_connect
-		(at 360.68 81.28)
-	)
 	(wire
 		(pts
@@
 	(wire
 		(pts
+			(xy 360.68 101.6) (xy 373.38 101.6)
+		)
+		(stroke
+			(width 0)
+			(type default)
+		)
+	)
+	(wire
+		(pts
 			(xy 360.68 152.4) (xy 369.57 152.4)
 		)
@@
 	(wire
 		(pts
+			(xy 360.68 81.28) (xy 370.84 81.28)
+		)
+		(stroke
+			(width 0)
+			(type default)
+		)
+	)
+	(wire
+		(pts
 			(xy 220.98 116.84) (xy 228.6 116.84)
 		)
@@
 	(wire
 		(pts
+			(xy 307.34 116.84) (xy 320.04 116.84)
+		)
+		(stroke
+			(width 0)
+			(type default)
+		)
+	)
+	(wire
+		(pts
 			(xy 347.98 60.96) (xy 345.44 60.96)
 		)
@@
 		(pts
 			(xy 254 77.47) (xy 255.27 77.47)
+		)
+		(stroke
+			(width 0)
+			(type default)
+		)
+	)
+	(wire
+		(pts
+			(xy 306.07 101.6) (xy 320.04 101.6)
+		)
+		(stroke
+			(width 0)
+			(type default)
+		)
+	)
+	(wire
+		(pts
+			(xy 360.68 99.06) (xy 373.38 99.06)
 		)
 		(stroke
@@
 		)
 	)
-	(label "TFT_MISO"
+	(label "TP_OUT"
 		(at 260.35 149.86 0)
 		(effects
@@
 		)
 	)
+	(label "USB_D+"
+		(at 373.38 101.6 0)
+		(effects
+			(font
+				(size 1.27 1.27)
+			)
+			(justify left bottom)
+		)
+	)
 	(label "RESET_STM_N"
 		(at 233.68 146.05 0)
@@
 		)
 	)
+	(label "AUDIO_IN"
+		(at 370.84 81.28 0)
+		(effects
+			(font
+				(size 1.27 1.27)
+			)
+			(justify left bottom)
+		)
+	)
 	(label "BTN_SELECT"
 		(at 307.34 109.22 0)
@@
 		)
 	)
-	(label "TFT_SCK"
+	(label "TP_CLK"
 		(at 260.35 144.78 0)
 		(effects
@@
 		)
 	)
+	(label "USB_D-"
+		(at 373.38 99.06 0)
+		(effects
+			(font
+				(size 1.27 1.27)
+			)
+			(justify left bottom)
+		)
+	)
 	(label "3V3_SYS"
 		(at 176.53 146.05 180)
@@
 		)
 	)
-	(label "TFT_MOSI"
+	(label "AUDIO_EN"
+		(at 307.34 116.84 0)
+		(effects
+			(font
+				(size 1.27 1.27)
+			)
+			(justify left bottom)
+		)
+	)
+	(label "TP_DIN"
 		(at 260.35 142.24 0)
 		(effects
@@
 		)
 	)
+	(label "Detection_USB"
+		(at 306.07 101.6 0)
+		(effects
+			(font
+				(size 1.27 1.27)
+			)
+			(justify left bottom)
+		)
+	)
